File: mirage/mirage.kicad_sch (KiCad schematic)
At the start: 9 parts, among them U1 STM32H573ZITx

Commit message: revert: remove testing
Other:
- note removed: "BA"
- note removed: "LOL"

Commit message: Updated silkscreen
Other:
- note added: "BA"
