File: mirage/connectors.kicad_sch (KiCad schematic)
At the start: 1 part, among them J1 MOLEX SL

Commit message: hi hello world world hello
Changed lines of the file:
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@@
 (kicad_sch
-	(version 20231120)
+	(version 20250114)
 	(generator "eeschema")
-	(generator_version "8.0")
+	(generator_version "9.0")
 	(paper "A4")
 	(wire
