File: mirage/untitled.kicad_sch (KiCad schematic)
At the start: 6 parts, among them U10 TPS62152RGTR

Commit message: feat: testing1
Parts:
- removed C20: 22uF, symbol Device:C_Small
- removed C21: 3.3nF, symbol Device:C_Small
- removed C22: 10uF, symbol Device:C_Small
- removed L1: 2.2uH, symbol Device:L_Small
- removed R4: 100k, symbol Device:R_Small
- removed U10: TPS62152RGTR, EasyEDA:TQFN-16_L3.0-W3.0-P0.50-TL-EP1.7, symbol EasyEDA:TPS62152RGTR
- added C23: 22uF, symbol Device:C_Small
- added C24: 10uF, symbol Device:C_Small
- added C25: 3.3nF, symbol Device:C_Small
- added L2: 2.2uH, symbol Device:L_Small
- added R5: 100k, symbol Device:R_Small
- added U11: TPS62152RGTR, EasyEDA:TQFN-16_L3.0-W3.0-P0.50-TL-EP1.7, symbol EasyEDA:TPS62152RGTR
Connections:
- net +3.3V: now also C23.2, L2.1, R5.1
- net BUCK_SW: now also L2.2, U11.1 (SW), U11.14 (VOS), U11.2 (SW), U11.3 (SW)
- net GND: now also C23.1, C24.2, C25.2, U11.15 (PGND), U11.16 (PGND), U11.5 (FB), U11.6 (AGND), U11.7 (FSW), U11.8 (DEF)
- net VBAT+: now also C24.1, U11.10 (AVIN), U11.11 (PVIN), U11.12 (PVIN)
- new net: R5.2, U11.4 (PG)
- new net: C25.1, U11.9 (SS/TR)
Other:
- company: (none) -> CUHAR

Commit message: hi hello world world hello
Changed lines of the file:
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@@
 (kicad_sch
-	(version 20231120)
+	(version 20250114)
 	(generator "eeschema")
-	(generator_version "8.0")
+	(generator_version "9.0")
 	(paper "A4")
 	(title_block
